File: PitotBoard2026/PitoBoard2026/PitoBoard2026.kicad_pcb (KiCad board)
At the start: 2 copper layers, 8.5 x 5.5 mm, 57 parts, among them J1 RJ25, J2 ICSP, J3 Conn_01x04_Socket, J4 Conn_01x04_Pin, SW1 RST, U1 ATmega328PB-A, U10 MCP25625-x-SS, U2 R-78E5.0-0.5, U4 SLIP, U6 SDP32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

Commit message: Add files via upload
Parts:
- removed D3: CLK, LED_SMD:LED_0603_1608Metric
- removed D4: PWR, LED_SMD:LED_0603_1608Metric
- removed R15, R16: 2.2k, Resistor_SMD:R_0603_1608Metric
- removed R7, R8: 1k, Resistor_SMD:R_0603_1608Metric
- added J5: Conn_01x04_Socket, Connector_PinSocket_2.54mm:PinSocket_1x04_P2.54mm_Vertical, F.Cu at (148.8, 40.2)
- added J6: Conn_01x04_Pin, Connector_PinHeader_2.54mm:PinHeader_1x04_P2.54mm_Horizontal, F.Cu at (90.6, 65.9)
- C3, D1, D2, D6, R17, R18, R20, R21, R22, R23: moved to B.Cu
- moved C14 181.0 mm to (221.3, 51.7), turned to -90 degrees
- moved U7 170.6 mm to (217.8, 51.8), turned to -90 degrees
- moved C15 164.8 mm to (214.1, 51.8), turned to -90 degrees
- moved J4 160.0 mm to (221.9, 58.9), turned to -90 degrees
- moved R12 135.3 mm to (219.8, 56.3), turned to 180 degrees
- moved R11 132.5 mm to (216.3, 56.3)
- moved J3 96.8 mm to (163.0, 44.1)
- moved J1 88.9 mm to (152.3, 72.0)
- moved D1 85.1 mm to (148.3, 78.0), turned to 90 degrees
- moved C1 84.2 mm to (159.1, 46.9), turned to 90 degrees
- moved U1 83.5 mm to (152.6, 47.4)
- moved U9 82.5 mm to (136.0, 64.4), turned to 180 degrees
- moved C16 82.5 mm to (159.6, 49.4), turned to 180 degrees
- moved C17 82.2 mm to (159.6, 50.9), turned to 180 degrees
- moved Y1 81.4 mm to (146.1, 50.9), turned to 90 degrees
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Connections:
- C27 pad 1: GND -> Net-(J6-Pin_2)
- C27 pad 2: +5V -> GND
- U1 pad 27: SDA0 -> SDA1
- U1 pad 28: SCL0 -> SCL1
- U1 pad 3: SDA1 -> SDA0
- U1 pad 6: SCL1 -> SCL0
- U6 pad 5: SCL0 -> Net-(J6-Pin_4)
- U6 pad 7: +5V -> Net-(J6-Pin_2)
- U6 pad 8: SDA0 -> Net-(J6-Pin_1)
Routing:
- net GND: track 0.00 -> 38.8 mm
- net RST: track 0.00 -> 30.4 mm, vias 0 -> 1
- net INT: track 0.00 -> 27.8 mm, vias 0 -> 2
- net SDA1: track 0.00 -> 25.8 mm, vias 0 -> 1
- net +5V: track 0.00 -> 23.9 mm, vias 0 -> 1
- net SCK: track 0.00 -> 23.9 mm, vias 0 -> 1
- net MISO: track 0.00 -> 22.3 mm, vias 0 -> 1
- net SCL1: track 0.00 -> 14.3 mm
- net +3V3: track 0.00 -> 12.1 mm
- net MOSI: track 0.00 -> 10.8 mm
- net Net-(U10-RXD): track 0.00 -> 7.70 mm
- net CS: track 0.00 -> 6.46 mm
- net Net-(U10-TXD): track 0.00 -> 6.08 mm, vias 0 -> 2
- net Net-(U7-VDD3V3): track 0.00 -> 5.46 mm
- net Net-(J6-Pin_4): track 0.00 -> 5.30 mm
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Other:
- board size 8.5 x 5.5 mm -> 8 x 5 mm

Commit message: 配線終わり(部品は違う)
Parts:
- moved C3 2.82 mm to (157.6, 73.4), turned to -90 degrees
- moved D2 2.30 mm to (161.8, 75.2)
- moved D1 1.82 mm to (146.5, 78.3)
- moved D6 1.00 mm to (136.3, 77.4)
Connections:
- J4 pad 1: GND -> GND1
Routing:
- net GND: track 38.8 -> 264.7 mm, vias 0 -> 2
- net +5V: track 23.9 -> 145.8 mm, vias 1 -> 4
- net Net-(D1-K): track 0.00 -> 38.3 mm
- net +3V3: track 12.1 -> 48.7 mm
- net GND1: track 0.00 -> 27.6 mm, vias 0 -> 3
- net SDA0: track 0.00 -> 27.0 mm, vias 0 -> 1
- net SCL0: track 0.00 -> 21.8 mm
- net CANH: track 0.00 -> 11.4 mm
- net CANL: track 0.00 -> 9.73 mm, vias 0 -> 2
- net SDA3: track 2.04 -> 11.0 mm
- net Net-(U1-~{RESET}/PC6): track 0.00 -> 8.52 mm, vias 0 -> 2
- net SCL3: track 0.00 -> 6.95 mm
- net Net-(D1-A): track 0.00 -> 6.55 mm
- net ERR: track 0.00 -> 6.12 mm, vias 0 -> 2
- net Net-(U10-VDDA): track 0.00 -> 5.32 mm
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