File: PitotBoard2026/PitoBoard2026/PitoBoard2026.kicad_sch (KiCad schematic)
At the start: 55 parts, among them J1 RJ25, J2 ICSP, J3 Conn_01x04_Socket, J4 Conn_01x04_Pin, SW1 RST, U1 ATmega328PB-A, U10 MCP25625-x-SS, U2 R-78E5.0-0.5, U4 SLIP, U6 SDP32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

Commit message: Add files via upload
Parts:
- removed D3: CLK, LED_SMD:LED_0603_1608Metric, symbol Device:LED
- removed D4: PWR, LED_SMD:LED_0603_1608Metric, symbol Device:LED
- removed R7, R8: 1k, Resistor_SMD:R_0603_1608Metric, symbol Device:R_US
- added J5: Conn_01x04_Socket, Connector_PinSocket_2.54mm:PinSocket_1x04_P2.54mm_Vertical, symbol Connector:Conn_01x04_Socket
- added J6: Conn_01x04_Pin, Connector_PinHeader_2.54mm:PinHeader_1x04_P2.54mm_Horizontal, symbol Connector:Conn_01x04_Pin
Connections:
- net +5V: now also J5.2 (Pin_2); no longer C27.2, U6.7 (VDD)
- net GND: now also C27.2, J5.3 (Pin_3), J6.3 (Pin_3); no longer C27.1
- net SCL0: now also U1.6 (PE1); no longer U1.28 (PC5), U6.5 (SCL)
- net SCL1: now also U1.28 (PC5), J5.4 (Pin_4); no longer U1.6 (PE1)
- net SDA0: now also U1.3 (PE0); no longer U1.27 (PC4), U6.8 (SDA)
- net SDA1: now also U1.27 (PC4), J5.1 (Pin_1); no longer U1.3 (PE0)
- new net: C27.1, J6.2 (Pin_2), U6.7 (VDD)
- new net: J6.4 (Pin_4), U6.5 (SCL)
- new net: J6.1 (Pin_1), U6.8 (SDA)
Other:
- note removed: "できるだけピンの近くに配置する。"
- note removed: "導通"
- moved on the sheet: C27

Commit message: 配線終わり(部品は違う)
Connections:
- net GND: no longer J4.1 (Pin_1)
- net GND1: now also J4.1 (Pin_1)
Changed lines of the file:
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@@
 			)
 		)
-		(property "Value" "GND"
+		(property "Value" "GND1"
 			(at 187.96 180.34 0)
 			(effects
