File: PitotBoard2026/PitoBoard2026.kicad_sch (KiCad schematic)
At the start: 57 parts, among them J1 RJ25, J2 ICSP, J3 Conn_01x04_Socket, J4 Conn_01x04_Pin, J5 Conn_01x04_Socket, J6 Conn_01x04_Pin, SW1 RST, U1 ATmega328PB-A, U10 MCP25625-x-SS, U2 AP7375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

Commit message: Add files via upload
Parts:
- C15, C5: footprint Capacitor_SMD:C_0805_2012Metric -> Capacitor_SMD:C_0603_1608Metric
- C3, C6, C7, C8, C9: footprint Capacitor_SMD:C_1206_3216Metric -> Capacitor_SMD:C_0603_1608Metric
Changed lines of the file:
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@@
 			)
 		)
-		(property "Footprint" "Capacitor_SMD:C_1206_3216Metric"
+		(property "Footprint" "Capacitor_SMD:C_0603_1608Metric"
 			(at 31.75 3.81 0)
 			(effects
@@
 			)
 		)
-		(property "Footprint" "Capacitor_SMD:C_1206_3216Metric"
+		(property "Footprint" "Capacitor_SMD:C_0603_1608Metric"
 			(at 52.07 3.81 0)
 			(effects
@@
 			)
 		)
-		(property "Footprint" "Capacitor_SMD:C_1206_3216Metric"
+		(property "Footprint" "Capacitor_SMD:C_0603_1608Metric"
 			(at 52.07 68.58 0)
 			(effects
@@
 			)
 		)
-		(property "Footprint" "Capacitor_SMD:C_0805_2012Metric"
+		(property "Footprint" "Capacitor_SMD:C_0603_1608Metric"
 			(at 232.41 173.99 0)
 			(effects
@@
 			)
 		)
-		(property "Footprint" "Capacitor_SMD:C_1206_3216Metric"
+		(property "Footprint" "Capacitor_SMD:C_0603_1608Metric"
 			(at 30.48 68.58 0)
 			(effects
@@
 			)
 		)
-		(property "Footprint" "Capacitor_SMD:C_1206_3216Metric"
+		(property "Footprint" "Capacitor_SMD:C_0603_1608Metric"
 			(at 25.4 68.58 0)
 			(effects
@@
 			)
 		)
-		(property "Footprint" "Capacitor_SMD:C_0805_2012Metric"
+		(property "Footprint" "Capacitor_SMD:C_0603_1608Metric"
 			(at 121.92 135.89 0)
 			(effects

Commit message: Add files via upload
Connections:
- net +5V: now also R11.1, R12.1
- net +5VA: no longer R11.1, R12.1
- net SCL0: now also J3.2 (Pin_2); no longer U4.7 (SCL)
- net SCL1: now also R12.2, U4.7 (SCL); no longer J3.2 (Pin_2)
- net SCL2: no longer R12.2
- net SDA0: now also J3.3 (Pin_3); no longer U4.6 (SDA)
- net SDA1: now also R11.2, U4.6 (SDA); no longer J3.3 (Pin_3)
- net SDA2: no longer R11.2
- net GND2: now reaches C27.2, J6.3 (Pin_3), U3.1 (GND), U3.10 (GND), U3.11 (GND), U3.2 (GND), U3.3 (GND), U3.6 (GND), U3.9 (ADDR)
- net GND2: now also U3.17 (GND1), U3.18 (GND1)
- no-connect marks 31 -> 29
Other:
- moved on the sheet: C4, C5, J2, J5, R11, R12, U4
