File: PitotBoard2026/PitotBoard2026.kicad_pcb (KiCad board)
At the start: 2 copper layers, 8 x 5 mm, 61 parts, among them J1 RJ25, J2 ICSP(, J3 Conn_01x04_Socket, J4 Conn_01x04_Pin, J5 Conn_01x04_Socket, J6 Conn_01x04_Pin, SW1 RST, U1 ATmega328PB-A, U10 MCP25625-x-SS, U11 FXMA2102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

Commit message: Add files via upload
Parts:
- U10: moved to B.Cu
- moved J1 150.3 mm to (164.1, 138.2)
- moved U9 123.5 mm to (171.7, 100.4)
- moved U3 120.5 mm to (152.9, 67.2), turned to 90 degrees
- moved U2 117.4 mm to (136.8, 132.9)
- moved J5 114.6 mm to (157.1, 89.4), turned to 90 degrees
- moved U10 110.3 mm to (158.9, 130.7), turned to 90 degrees
- moved J6 108.8 mm to (157.6, 63.3)
- moved U11 104.1 mm to (157.4, 96.9)
- moved U5 98.0 mm to (139.3, 117.5)
- moved U1 97.3 mm to (150.8, 97.3)
Other:
- board size 8 x 5 mm -> 5 x 8 mm

Commit message: Add files via upload
Parts:
- C1, C24, C6, C7, D6, R9, U1, U2, U5, Y1, Y3: moved to B.Cu
- moved C14 184.1 mm to (194.3, 133.7), turned to 180 degrees
- moved C15 182.6 mm to (191.6, 137.9), turned to -90 degrees
- moved J4 181.4 mm to (202.3, 133.4)
- moved C3 169.4 mm to (169.4, 134.6)
- moved C9 168.2 mm to (169.4, 133.1)
- moved C10 165.9 mm to (169.4, 131.6)
- moved C8 165.4 mm to (173.0, 133.9), turned to -90 degrees
- moved C12 164.4 mm to (172.9, 128.7)
- moved C11 163.6 mm to (169.4, 130.1)
- moved C7 158.4 mm to (174.2, 113.7)
- moved R9 154.4 mm to (161.5, 136.2)
- moved C6 154.2 mm to (167.8, 114.9), turned to 180 degrees
- moved C21 153.2 mm to (162.1, 130.8), turned to 180 degrees
- moved C2 152.9 mm to (159.7, 116.7), turned to 90 degrees
- moved C22 152.7 mm to (162.1, 132.3), turned to 180 degrees
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Connections:
- U10 pad 26: unconnected-(U10-VSS-Pad26) -> GND
Routing:
- net CANH: track 0.00 -> 8.68 mm, vias 0 -> 1
- net Net-(U10-RXD): track 0.00 -> 6.65 mm
- net Net-(U10-TXD): track 0.00 -> 4.82 mm
- net CANL: track 0.00 -> 4.30 mm
- net GND: track 0.00 -> 2.34 mm, vias 0 -> 1
- net Net-(D1-A): track 0.00 -> 2.18 mm
- net Net-(U1-AREF): track 0.00 -> 1.98 mm
- net +5V: track 0.00 -> 1.17 mm, vias 0 -> 1

Commit message: Add files via upload
Parts:
- C27, C4, R11, R12, R20, R21, R22, R23: moved to B.Cu
- moved R22 149.1 mm to (172.6, 122.1)
- moved R20 147.9 mm to (169.3, 120.0), turned to 180 degrees
- moved R21 147.7 mm to (169.3, 122.1), turned to 180 degrees
- moved R23 146.7 mm to (172.6, 120.0)
- moved C4 139.7 mm to (149.2, 113.7), turned to -90 degrees
- moved C5 136.5 mm to (147.2, 113.2), turned to -90 degrees
- moved R11 131.6 mm to (153.4, 113.3)
- moved R12 129.5 mm to (153.4, 111.8)
- moved C27 116.3 mm to (136.8, 112.2)
- moved J4 69.5 mm to (132.8, 131.7), turned to 90 degrees
- moved C14 61.4 mm to (133.0, 137.2), turned to 90 degrees
- moved U7 59.6 mm to (136.5, 137.3), turned to 90 degrees
- moved C15 54.6 mm to (137.1, 141.8), turned to 0 degrees
- moved J6 52.1 mm to (133.2, 109.3), turned to 90 degrees
- moved U3 50.1 mm to (137.0, 114.7), turned to 180 degrees
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Routing:
- net GND: track 2.34 -> 156.1 mm, vias 1 -> 6
- net +5V: track 1.17 -> 126.4 mm, vias 1 -> 5
- net +3V3: track 0.00 -> 58.0 mm, vias 0 -> 1
- net INT: track 0.00 -> 32.5 mm, vias 0 -> 2
- net GND2: track 0.00 -> 26.9 mm, vias 0 -> 1
- net SDA0: track 0.00 -> 25.7 mm, vias 0 -> 1
- net SCL0: track 0.00 -> 24.9 mm
- net SDA3: track 0.00 -> 21.5 mm
- net GND1: track 0.00 -> 19.9 mm
- net SCL3: track 0.00 -> 18.3 mm, vias 0 -> 1
- net SCK: track 0.00 -> 16.6 mm, vias 0 -> 1
- net RST: track 0.00 -> 15.9 mm
- net +5VA: track 0.00 -> 15.9 mm, vias 0 -> 2
- net Net-(D1-K): track 0.00 -> 14.8 mm
- net MOSI: track 0.00 -> 12.9 mm, vias 0 -> 2
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Other:
- board size 5 x 8 mm -> 49.4 x 41 mm

Commit message: Add files via upload
Parts:
- added REF**: MountingHole_2.2mm_M2, MountingHole:MountingHole_2.2mm_M2, F.Cu at (177.3, 146.4)
- added REF**: MountingHole_2.2mm_M2, MountingHole:MountingHole_2.2mm_M2, F.Cu at (141.0, 143.2)
- added REF**: MountingHole_2.2mm_M2, MountingHole:MountingHole_2.2mm_M2, F.Cu at (149.2, 146.4)
- added REF**: MountingHole_2.2mm_M2, MountingHole:MountingHole_2.2mm_M2, F.Cu at (132.7, 143.2)
- moved J1 0.10 mm to (164.1, 138.3)
Routing:
- net GND: track 156.1 -> 155.3 mm, vias 6 -> 35
- net GND2: vias 1 -> 2
- net GND1: vias 0 -> 3
- added copper zone on B.Cu, net GND
- added copper zone on F.Cu, net GND
- added copper zone on B.Cu, net GND1
- added copper zone on F.Cu, net GND1
- added copper zone on B.Cu, net GND2
- added copper zone on F.Cu, net GND2
Other:
- board size 49.4 x 41 mm -> 50.2 x 41.5 mm
